Commit message: jhbdf

File: Gantry.urdf (robot description, URDF)
Before this commit: robot gantry, 1 links, 0 joints
Links:
- added link gimbal_frame_link, mass 2; collision box size=0.1 0.1 0.1; visual box size=0.1 0.1 0.1
- added link leg1_link, mass 2; collision box size=0.05 0.05 0.4; visual box size=0.05 0.05 0.4
- added link leg2_link, mass 2; collision box size=0.05 0.05 0.4; visual box size=0.05 0.05 0.4
- added link leg3_link, mass 2; collision box size=0.05 0.05 0.4; visual box size=0.05 0.05 0.4
- added link leg4_link, mass 2; collision box size=0.05 0.05 0.4; visual box size=0.05 0.05 0.4
- added link upperFrame1_link, mass 2; collision box size=0.05 0.85 0.05; visual box size=0.05 0.85 0.05
- added link upperFrame2_link, mass 2; collision box size=0.05 0.85 0.05; visual box size=0.05 0.85 0.05
- added link upperFrame3_link, mass 2; collision box size=1.55 0.05 0.05; visual box size=1.55 0.05 0.05
- added link upperFrame4_link, mass 2; collision box size=1.55 0.05 0.05; visual box size=1.55 0.05 0.05
- added link world
- added link yaxis_link, mass 2; collision box size=0.1 0.85 0.1; visual box size=0.1 0.85 0.1
- added link zaxis_link, mass 2; collision box size=0.1 0.1 0.8; visual box size=0.1 0.1 0.8
- link base_link: mass None -> 12; geometry collision box size=2.5 1.5 0.05; visual box size=2.5 1.5 0.05
Joints:
- added joint base_joint: type fixed, parent world, child base_link, origin xyz=0 0 0.05 rpy=0 0 0
- added joint gimbal_frame_sliding_joint: type prismatic, parent zaxis_link, child gimbal_frame_link, origin xyz=0.1 0 0 rpy=0 0 0, axis 0 0 1, limit lower=-0.35 upper=0.35 effort=100 velocity=100
- added joint leg1_joint: type fixed, parent base_link, child leg1_link, origin xyz=0.75 0.4 0.2 rpy=0 0 0
- added joint leg2_joint: type fixed, parent base_link, child leg2_link, origin xyz=0.75 -0.4 0.2 rpy=0 0 0
- added joint leg3_joint: type fixed, parent base_link, child leg3_link, origin xyz=-0.75 0.4 0.2 rpy=0 0 0
- added joint leg4_joint: type fixed, parent base_link, child leg4_link, origin xyz=-0.75 -0.4 0.2 rpy=0 0 0
- added joint upperFrame1_joint: type fixed, parent base_link, child upperFrame1_link, origin xyz=-0.75 0 0.375 rpy=0 0 0
- added joint upperFrame2_joint: type fixed, parent base_link, child upperFrame2_link, origin xyz=0.75 0 0.375 rpy=0 0 0
- added joint upperFrame3_joint: type fixed, parent base_link, child upperFrame3_link, origin xyz=0 0.4 0.375 rpy=0 0 0
- added joint upperFrame4_joint: type fixed, parent base_link, child upperFrame4_link, origin xyz=0 -0.4 0.375 rpy=0 0 0
- added joint yaxis_sliding_joint: type prismatic, parent upperFrame1_link, child yaxis_link, origin xyz=0.025 0 0.075 rpy=0 0 0, axis 1 0 0, limit lower=0 upper=1.2 effort=100 velocity=100
- added joint zaxis_sliding_joint: type prismatic, parent yaxis_link, child zaxis_link, origin xyz=0.1 0 0 rpy=0 0 0, axis 0 1 0, limit lower=-0.3 upper=0.3 effort=100 velocity=100
