Commit message: nn

File: Gantry_CAD.urdf (robot description, URDF)
Before this commit: robot Gantry_CAD, 5 links, 4 joints
Links:
- removed link gimbal_holder_link
- added link gimbal_interface_link, mass 1.0; collision box size=1 1 1; visual mesh filename=GIMBAL_INTERFACE.STL scale=0.001 0.001 0.001
- link base_link: geometry collision box size=1 1 1; visual mesh filename=GANTRY_FRAME.STL scale=0.001 0.001 0.001
Joints:
- removed joint gimbal_holder_joint
- added joint gimbal_interface_joint: type prismatic, parent zaxis_link, child gimbal_interface_link, origin xyz=0.004 0.4 0 rpy=0 0 0, axis 0 1 0, limit lower=-0.39 upper=0.4 effort=100 velocity=100
- joint yaxis_joint: limit lower=0 upper=1.35 effort=100 velocity=100 -> lower=0 upper=1.2 effort=100 velocity=100; origin xyz=0.3 0.47 -0.4 rpy=0 0 0 -> xyz=0.289 0.4695 -0.19 rpy=0 0 0
- joint zaxis_joint: limit lower=-0.35 upper=0.35 effort=100 velocity=100 -> lower=-0.34 upper=0.34 effort=100 velocity=100; origin xyz=0.45 -0.4 0 rpy=0 0 0 -> xyz=0.47 -0.416 -0.007 rpy=0 0 0

Commit message: ewg

File: Gantry_CAD.urdf (robot description, URDF)
Before this commit: robot Gantry_CAD, 5 links, 4 joints
Links:
- added link pitch_axis_link, mass 1.0; collision box size=1 1 1; visual mesh filename=PITCHAXIS.STL scale=0.001 0.001 0.001
- added link roll_axis_link, mass 1.0; collision box size=1 1 1; visual mesh filename=ROLLAXIS.STL scale=0.001 0.001 0.001
- added link yaw_axis_link, mass 1.0; collision box size=1 1 1; visual mesh filename=YAWAXIS.STL scale=0.001 0.001 0.001
Joints:
- added joint pitch_axis_joint: type revolute, parent yaw_axis_link, child pitch_axis_link, origin xyz=0 0 0 rpy=0 0 0, axis 0 1 0, limit lower=-1.570796327 upper=1.570796327 effort=100 velocity=2
- added joint roll_axis_joint: type fixed, parent pitch_axis_link, child roll_axis_link, origin xyz=0 0 0 rpy=0 0 0
- added joint yaw_axis_joint: type fixed, parent gimbal_interface_link, child yaw_axis_link, origin xyz=-1.209 -0.692 1.451 rpy=0 1.570796327 0
- joint yaxis_joint: limit lower=0 upper=1.2 effort=100 velocity=100 -> lower=0 upper=1.1 effort=100 velocity=100

Commit message: knl

File: Gantry_CAD.urdf (robot description, URDF)
Before this commit: robot Gantry_CAD, 8 links, 7 joints
Links:
- added link end_eff_interface_link, mass 1.0; collision box size=1 1 1; visual mesh filename=END_EFF_INTERFACE.STL scale=0.001 0.001 0.001
Joints:
- added joint end_eff_interface_joint: type fixed, parent roll_axis_link, child end_eff_interface_link, origin xyz=0.57 1 1.253 rpy=0 0 -1.570796327
- joint base_joint: origin xyz=-0.00316703 -0.01282036 -0.00465 rpy=1.570796327 0 1.570796327 -> xyz=0 0 0 rpy=1.570796327 0 1.570796327
- joint gimbal_interface_joint: origin xyz=0.004 0.4 0 rpy=0 0 0 -> xyz=0 -0.36733 0.117 rpy=0 0 0
- joint pitch_axis_joint: origin xyz=0 0 0 rpy=0 0 0 -> xyz=-0.177 0.0155 -0.0125 rpy=0 0 0
- joint roll_axis_joint: origin xyz=0 0 0 rpy=0 0 0 -> xyz=-0.59 -0.82 -1.2 rpy=0 0 0
- joint yaw_axis_joint: origin xyz=-1.209 -0.692 1.451 rpy=0 1.570796327 0 -> xyz=0.002 -0.055 0 rpy=0 1.570796327 0
- joint yaxis_joint: origin xyz=0.289 0.4695 -0.19 rpy=0 0 0 -> xyz=0.28605 0.515 0.84441 rpy=0 0 0
- joint zaxis_joint: origin xyz=0.47 -0.416 -0.007 rpy=0 0 0 -> xyz=0.40184 0.5385 0.042 rpy=0 0 0

Commit message: fm

File: Gantry_CAD.urdf (robot description, URDF)
Before this commit: robot Gantry_CAD, 9 links, 8 joints
Joints:
- joint end_eff_interface_joint: axis (none) -> 0 1 0; limit (none) -> lower=-3.141592654 upper=3.141592654 effort=100 velocity=2; origin xyz=0.57 1 1.253 rpy=0 0 -1.570796327 -> xyz=-0.0374949 0.0006177 0.0715 rpy=0 0 -1.570796327; type fixed -> revolute
- joint gimbal_interface_joint: limit lower=-0.39 upper=0.4 effort=100 velocity=100 -> lower=-0.4 upper=0.33 effort=100 velocity=100
- joint pitch_axis_joint: limit lower=-1.570796327 upper=1.570796327 effort=100 velocity=2 -> lower=-3.141592654 upper=3.141592654 effort=100 velocity=2; origin xyz=-0.177 0.0155 -0.0125 rpy=0 0 0 -> xyz=-0.155 0.0205 0.0625 rpy=0 0 0
- joint roll_axis_joint: axis (none) -> 0 0 1; limit (none) -> lower=-1.570796327 upper=1.570796327 effort=100 velocity=2; origin xyz=-0.59 -0.82 -1.2 rpy=0 0 0 -> xyz=0 0.147789 -0.0715 rpy=0 0 0; type fixed -> revolute
- joint yaxis_joint: limit lower=0 upper=1.1 effort=100 velocity=100 -> lower=0 upper=1 effort=100 velocity=100; origin xyz=0.28605 0.515 0.84441 rpy=0 0 0 -> xyz=0.28605 0.515 0.35 rpy=0 0 0
- joint zaxis_joint: limit lower=-0.34 upper=0.34 effort=100 velocity=100 -> lower=-0.24 upper=0.34 effort=100 velocity=100

Commit message: 4h5

File: Gantry_CAD.urdf (robot description, URDF)
Before this commit: robot Gantry_CAD, 9 links, 8 joints
Links:
- added link end_eff_link, mass 1.0; collision mesh filename=END_EFF.STL scale=0.001 0.001 0.001; visual mesh filename=END_EFF.STL scale=0.001 0.001 0.001
- added link target_frame_link, mass 1.0; collision mesh filename=TARGET_FRAME.STL scale=0.001 0.001 0.001; visual mesh filename=TARGET_FRAME.STL scale=0.001 0.001 0.001
- link base_link: geometry collision mesh filename=GANTRY_FRAME.STL scale=0.001 0.001 0.001; visual mesh filename=GANTRY_FRAME.STL scale=0.001 0.001 0.001
Joints:
- added joint end_eff_joint: type fixed, parent end_eff_interface_link, child end_eff_link, origin xyz=0 -0.053 0 rpy=0 -1.570796327 3.14159265359
- added joint target_frame_joint: type fixed, parent base_link, child target_frame_link, origin xyz=1.01205 0.485 1.8327 rpy=0 3.14159265359 0
- joint gimbal_interface_joint: limit lower=-0.4 upper=0.33 effort=100 velocity=100 -> lower=0.15 upper=0.902 effort=100 velocity=100; origin xyz=0 -0.36733 0.117 rpy=0 0 0 -> xyz=0 -0.96491 0.117 rpy=0 0 0
- joint pitch_axis_joint: limit lower=-3.141592654 upper=3.141592654 effort=100 velocity=2 -> lower=-1.39626340159546 upper=1.39626340159546 effort=100 velocity=2
- joint roll_axis_joint: limit lower=-1.570796327 upper=1.570796327 effort=100 velocity=2 -> lower=-1.48352986419518 upper=1.48352986419518 effort=100 velocity=2
- joint yaxis_joint: limit lower=0 upper=1 effort=100 velocity=100 -> lower=0.038 upper=1.35 effort=100 velocity=100; origin xyz=0.28605 0.515 0.35 rpy=0 0 0 -> xyz=0.28605 0.515 0.3227 rpy=0 0 0
- joint zaxis_joint: limit lower=-0.24 upper=0.34 effort=100 velocity=100 -> lower=-0.72 upper=-0.12 effort=100 velocity=100; origin xyz=0.40184 0.5385 0.042 rpy=0 0 0 -> xyz=0.882 0.5385 0.042 rpy=0 0 0
